Commit message: plugin missile control able to get data from joystick

File: src/exocet_mm40_description/urdf/exocetMM40.xacro (robot description, xacro)
@@ -284,4 +284,6 @@
   </collision>
 </link>
+<!-- <xacro:property name="fins_limit_absolute" value="0.785398" /> -->
+<xacro:property name="fins_limit_absolute" value="0.349066" />
 <joint name="fins_fold1" type="revolute">
   <origin xyz="-0.04273 0.042755 0.0" rpy="0 0 0"/>
@@ -296,5 +298,5 @@
   <child link="FinHolder_1"/>
   <axis xyz="-0.707107 0.707107 -0.0"/>
-  <limit upper="0.349066" lower="-0.349066" effort="100" velocity="100"/>
+  <limit upper="${fins_limit_absolute}" lower="${-1*fins_limit_absolute}" effort="100" velocity="100"/>
 </joint>
 <joint name="fins_fold2" type="revolute">
@@ -310,5 +312,5 @@
   <child link="FinHolder_4"/>
   <axis xyz="-0.707107 -0.707107 -0.0"/>
-  <limit upper="0.349066" lower="-0.349066" effort="100" velocity="100"/>
+  <limit upper="${fins_limit_absolute}" lower="${-1*fins_limit_absolute}" effort="100" velocity="100"/>
 </joint>
 <joint name="fins_fold3" type="revolute">
@@ -324,5 +326,5 @@
   <child link="FinHolder_3"/>
   <axis xyz="0.707107 -0.707107 0.0"/>
-  <limit upper="0.349066" lower="-0.349066" effort="100" velocity="100"/>
+  <limit upper="${fins_limit_absolute}" lower="${-1*fins_limit_absolute}" effort="100" velocity="100"/>
 </joint>
 <joint name="fins_fold4" type="revolute">
@@ -338,5 +340,5 @@
   <child link="FinHolder_2"/>
   <axis xyz="0.707107 0.707107 0.0"/>
-  <limit upper="0.349066" lower="-0.349066" effort="100" velocity="100"/>
+  <limit upper="${fins_limit_absolute}" lower="${-1*fins_limit_absolute}" effort="100" velocity="100"/>
 </joint>
 <joint name="wings_fold1" type="revolute">
